Commit message: new file:   hector_quadrotor/hector_quadrotor_demo/launch/outdoor_flight_gazebo_asus.launch 	modified:   hector_quadrotor/hector_quadrotor_demo/launch/outdoor_flight_gazebo_dw_cam.launch 	new file:   hector_quadrotor/hector_quadrotor_demo/rviz_cfg/outdoor_flight_asus_cam.rviz 	new file:   hector_quadrotor/hector_quadrotor_demo/rviz_cfg/outdoor_flight_dw_cam.rviz 	modified:   hector_quadrotor/hector_quadrotor_description/urdf/quadrotor_with_asus.urdf.xacro

File: hector_quadrotor/hector_quadrotor_description/urdf/quadrotor_with_asus.urdf.xacro (robot description, xacro)
@@ -9,5 +9,5 @@
     <xacro:include filename="$(find hector_sensors_description)/urdf/asus_camera.urdf.xacro" />
     <xacro:asus_camera name="camera" parent="base_link">
-      <origin xyz="0.1 0.0 -0.03" rpy="0 ${M_PI/9} 0"/>
+      <origin xyz="0.1 0.0 -0.03" rpy="0 ${M_PI/2} 0"/>
     </xacro:asus_camera>
 </robot>
